File: EmisorASV/EmisorASV.kicad_sch (KiCad schematic)
At the start: 12 parts, among them J1 USB_C_Receptacle_USB2.0_16P, U1 ESP32ASV

Commit message: Agrega diseños del emisor y receptor LoRa ASV con documentación y fabricación
Parts:
- removed C1, C3: 10u, symbol Device:C
- removed C2, C4, C6: 100n, symbol Device:C
- removed J1: USB_C_Receptacle_USB2.0_16P, symbol Connector:USB_C_Receptacle_USB2.0_16P
- removed J_ANT: Conn_01x01_Pin, Connector_Wire:SolderWire-1.5sqmm_1x01_D1.7mm_OD3mm, symbol Connector:Conn_01x01_Pin
- removed LORA1: (no value), Oscillator:Oscillator_SMD_Abracon_ASV-4Pin_7.0x5.1mm, symbol ASV_Custom:XL1278_SMT_Module
- removed U1: ESP32ASV, ESP32-DEVKITC-32UE:ESPRESSIF_ESP32-DEVKITC-32UE, symbol ESP32-DEVKITC-32UE:ESP32ASV
- added C4: 47u / 25 V, Capacitor_THT:CP_Radial_D5.0mm_P2.00mm, symbol Device:C_Polarized
- added C6: 22u / 25 V, Capacitor_THT:CP_Radial_D5.0mm_P2.00mm, symbol Device:C_Polarized
- added C7: 100n / 50 V, Capacitor_THT:C_Disc_D5.0mm_W2.5mm_P5.00mm, symbol Device:C
- added C8: 10u / 25 V, Capacitor_THT:CP_Radial_D5.0mm_P2.00mm, symbol Device:C_Polarized
- added J4: SMA FUTURO - NO MONTAR, Connector_Coaxial:SMA_Amphenol_132134_Vertical, symbol Connector:Conn_Coaxial
- added JP2: ABIERTO con resorte, Connector_PinHeader_2.54mm:PinHeader_1x02_P2.54mm_Vertical, symbol Jumper:Jumper_2_Open
- added U2: LD1117V33 / 3,3 V LoRa, Package_TO_SOT_THT:TO-220-3_Vertical, symbol ASV_Emisor:LD1117V33_TO220
- added U3: ESP32-DEVKITC-32UE, ASV_Emisor:ESPRESSIF_ESP32-DEVKITC-32UE, symbol ASV_Emisor:ESP32_DEVKITC_32UE
- added U4: LoRa SX1278 / 433 MHz, ASV_Emisor:XL1278_SMT_16P_16.5x17mm_P1.27mm, symbol ASV_Emisor:XL1278_SMT_433_VERIFICAR
- C5: value 10u -> 100n / 50 V; footprint (none) -> Capacitor_THT:C_Disc_D5.0mm_W2.5mm_P5.00mm
- R1, R2: value 5.1k -> 10k; footprint (none) -> Resistor_THT:R_Axial_DIN0207_L6.3mm_D2.5mm_P7.62mm_Horizontal
Connections:
- net GND: now also C4.2, C6.2, C7.2, C8.2, J4.2 (Ext), U2.1 (GND), U3.14 (GND), U3.20 (GND), U3.26 (GND), U4.1 (GND), U4.12 (GND), U4.15 (GND RF); no longer R1.2, R2.2
- net LORA_DIO0: now also U3.10 (26 / DIO0), U4.10 (DIO0)
- net LORA_NSS: now also R1.2, U3.11 (27 / NSS), U4.9 (NSS)
- net LORA_3V3: now reaches R1.1
- net LORA_3V3: now also R2.1, C6.1, C7.1, C8.1, U2.2 (OUT), U4.5 (VCC 3V3)
- net SYS_5V: now reaches C5.1
- net SYS_5V: now also C4.1, U2.3 (IN), U3.19 (5V)
- new net LORA_DIO1: U3.9 (25 / DIO1), U4.2 (DIO1)
- new net LORA_DIO2: U3.8 (33 / DIO2), U4.3 (DIO2)
- new net LORA_MISO: U3.27 (19 / MISO), U4.6 (MISO)
- new net LORA_MOSI: U3.21 (23 / MOSI), U4.7 (MOSI)
- new net LORA_RESET: R2.2, U3.12 (14 / RESET), U4.11 (RESET)
- new net LORA_SCK: U3.28 (18 / SCK), U4.8 (SCK)
- new net RF_433: JP2.1 (A), U4.16 (ANT)
- new net RF_SMA: J4.1 (In), JP2.2 (B)
- no-connect marks 9 -> 29
Other:
- note added: "EMISOR ASV - ESP32 + LoRa 433 MHz"
- note added: "El celular debe funcionar como host USB OTG y suministrar energia. No aplicar 12 V ni tension de bateria al DevKit. Sin borneras UART. R1/R2: pull-ups NSS y RESET. C5/C6 junto a U2; C7/C8 junto al radio. Antena actual: resorte. No montar J4/JP2; ANT no va a GND. Punto = union; cruce sin punto = cables separados."
- note added: "USB DEL DEVKIT = ENTRADA DE ALIMENTACION 5 V"
- note added: "USB del celular al DevKit. Solo LoRa SMD; resto THT."
- company: (none) -> UCC - ASV
- title: (none) -> ASV - Emisor LoRa 433 MHz
