File: EmisorASV/EmisorASV.kicad_pcb (KiCad board)
At the start: 2 copper layers, 95 x 80 mm, 18 parts, among them J4 SMA FUTURO - NO MONTAR, U2 LD1117V33 / 3,3 V LoRa, U3 ESP32-DEVKITC-32UE, U4 LoRa SX1278 / 433 MHz

Commit message: puto
Routing:
- net /SYS_5V: track 205.4 -> 150.4 mm
- net /GND: track 246.7 -> 231.5 mm
- net /LORA_NSS: track 36.9 -> 37.7 mm
- net /LORA_DIO0: track 42.6 -> 43.2 mm

Commit message: emisor creo q esta listo, vr el tema usb c
Routing:
- net /LORA_MISO: track 89.4 -> 90.5 mm
- net /LORA_SCK: track 65.1 -> 65.9 mm
Changed lines of the file:
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@@
-	)
-	(segment
-		(start 100 48.14)
-		(end 96.7 48.14)
-		(width 0.5)
-		(layer "B.Cu")
-		(net "/GND")
 	)
 	(segment
@@
 	)
 	(segment
-		(start 96.7 63.38)
-		(end 89.08 63.38)
-		(width 0.7)
-		(layer "B.Cu")
-		(net "/GND")
-	)
-	(segment
 		(start 91.3197 46.3125)
 		(end 93.1472 48.14)
@@
 	)
 	(segment
-		(start 89.08 63.38)
-		(end 71.3 81.16)
-		(width 0.7)
+		(start 101.5 77)
+		(end 101.5 51)
+		(width 0.5)
 		(layer "B.Cu")
 		(net "/GND")
@@
 	)
 	(segment
-		(start 100 79.89)
-		(end 100 48.14)
-		(width 0.5)
+		(start 88.96 63.5)
+		(end 71.3 81.16)
+		(width 0.7)
+		(layer "B.Cu")
+		(net "/GND")
+	)
+	(segment
+		(start 96.7 63.38)
+		(end 96.58 63.5)
+		(width 0.7)
 		(layer "B.Cu")
 		(net "/GND")
@@
 	)
 	(segment
-		(start 74 79.89)
-		(end 100 79.89)
-		(width 0.5)
-		(layer "B.Cu")
-		(net "/GND")
-	)
-	(segment
 		(start 64 93)
 		(end 64 88.46)
@@
 	)
 	(segment
+		(start 98.64 48.14)
+		(end 96.7 48.14)
+		(width 0.5)
+		(layer "B.Cu")
+		(net "/GND")
+	)
+	(segment
+		(start 54.54 45.46)
+		(end 54.54 37)
+		(width 0.7)
+		(layer "B.Cu")
+		(net "/GND")
+	)
+	(segment
+		(start 54.08 46.08)
+		(end 54.08 50)
+		(width 0.7)
+		(layer "B.Cu")
+		(net "/GND")
+	)
+	(segment
+		(start 98.61 79.89)
+		(end 101.5 77)
+		(width 0.5)
+		(layer "B.Cu")
+		(net "/GND")
+	)
+	(segment
+		(start 52.3424 35.1719)
+		(end 54.2211 37.0505)
+		(width 0.7)
+		(layer "B.Cu")
+		(net "/GND")
+	)
+	(segment
+		(start 33.3827 54.3)
+		(end 32.1127 55.57)
+		(width 0.7)
+		(layer "B.Cu")
+		(net "/GND")
+	)
+	(segment
+		(start 51.127 35.1719)
+		(end 52.3424 35.1719)
+		(width 0.7)
+		(layer "B.Cu")
+		(net "/GND")
+	)
+	(segment
 		(start 71.3 81.16)
 		(end 74 79.89)
@@
 	)
 	(segment
-		(start 54.54 45.46)
-		(end 54.54 37)
-		(width 0.7)
-		(layer "B.Cu")
-		(net "/GND")
-	)
-	(segment
-		(start 54.08 46.08)
-		(end 54.08 50)
-		(width 0.7)
-		(layer "B.Cu")
-		(net "/GND")
-	)
-	(segment
-		(start 52.3424 35.1719)
-		(end 54.2211 37.0505)
-		(width 0.7)
-		(layer "B.Cu")
-		(net "/GND")
-	)
-	(segment
-		(start 33.3827 54.3)
-		(end 32.1127 55.57)
-		(width 0.7)
-		(layer "B.Cu")
-		(net "/GND")
-	)
-	(segment
-		(start 51.127 35.1719)
-		(end 52.3424 35.1719)
+		(start 96.58 63.5)
+		(end 88.96 63.5)
 		(width 0.7)
 		(layer "B.Cu")
@@
 	)
 	(segment
+		(start 74 79.89)
+		(end 98.61 79.89)
+		(width 0.5)
+		(layer "B.Cu")
+		(net "/GND")
+	)
+	(segment
 		(start 33.54 31.46)
 		(end 36.1298 34.0498)
@@
 	)
 	(segment
+		(start 101.5 51)
+		(end 98.64 48.14)
+		(width 0.5)
+		(layer "B.Cu")
+		(net "/GND")
+	)
+	(segment
 		(start 50.0049 34.0498)
 		(end 51.127 35.1719)
@@
 	)
 	(segment
+		(start 50.85 60.65)
+		(end 57.01 54.49)
+		(width 0.5)
+		(layer "B.Cu")
+		(net "/LORA_MISO")
+	)
+	(segment
 		(start 75.4044 54.49)
 		(end 80.4844 49.41)
@@
 	)
 	(segment
-		(start 50.85 60.65)
-		(end 57.01 54.49)
-		(width 0.5)
-		(layer "B.Cu")
-		(net "/LORA_MISO")
-	)
-	(segment
-		(start 98.675 50.8178)
-		(end 98.675 68.3216)
+		(start 95.3592 67.2608)
+		(end 96.7 65.92)
+		(width 0.5)
+		(layer "B.Cu")
+		(net "/LORA_MISO")
+	)
+	(segment
+		(start 80.4844 49.41)
+		(end 97.2672 49.41)
 		(width 0.5)
 		(layer "B.Cu")
@@
 	)
 	(segment
-		(start 80.4844 49.41)
-		(end 97.2672 49.41)
+		(start 39.785 60.65)
+		(end 50.85 60.65)
+		(width 0.5)
+		(layer "B.Cu")
+		(net "/LORA_MISO")
+	)
+	(segment
+		(start 100 52.1428)
+		(end 100 66.9966)
+		(width 0.5)
+		(layer "B.Cu")
+		(net "/LORA_MISO")
+	)
+	(segment
+		(start 57.01 54.49)
+		(end 75.4044 54.49)
+		(width 0.5)
+		(layer "B.Cu")
+		(net "/LORA_MISO")
+	)
+	(segment
+		(start 96.1457 69.7285)
+		(end 95.3592 68.942)
+		(width 0.5)
+		(layer "B.Cu")
+		(net "/LORA_MISO")
+	)
+	(segment
+		(start 100 66.9966)
+		(end 97.2681 69.7285)
+		(width 0.5)
+		(layer "B.Cu")
+		(net "/LORA_MISO")
+	)
+	(segment
+		(start 97.2672 49.41)
+		(end 100 52.1428)
 		(width 0.5)
 		(layer "B.Cu")
@@
 	)
 	(segment
-		(start 98.675 68.3216)
-		(end 97.2681 69.7285)
-		(width 0.5)
-		(layer "B.Cu")
-		(net "/LORA_MISO")
-	)
-	(segment
-		(start 97.2672 49.41)
-		(end 98.675 50.8178)
-		(width 0.5)
-		(layer "B.Cu")
-		(net "/LORA_MISO")
-	)
-	(segment
-		(start 96.1457 69.7285)
-		(end 95.3592 68.942)
-		(width 0.5)
-		(layer "B.Cu")
-		(net "/LORA_MISO")
-	)
-	(segment
-		(start 39.785 60.65)
-		(end 50.85 60.65)
-		(width 0.5)
-		(layer "B.Cu")
-		(net "/LORA_MISO")
-	)
-	(segment
-		(start 95.3592 67.2608)
-		(end 96.7 65.92)
-		(width 0.5)
-		(layer "B.Cu")
-		(net "/LORA_MISO")
-	)
-	(segment
-		(start 57.01 54.49)
-		(end 75.4044 54.49)
-		(width 0.5)
-		(layer "B.Cu")
-		(net "/LORA_MISO")
-	)
-	(segment
-		(start 97.9517 62.8444)
-		(end 97.9517 67.2083)
+		(start 99 66.16)
+		(end 96.7 68.46)
 		(width 0.5)
 		(layer "B.Cu")
@@
 	)
 	(segment
+		(start 59.4141 62.11)
+		(end 97.2173 62.11)
+		(width 0.5)
+		(layer "B.Cu")
+		(net "/LORA_SCK")
+	)
+	(segment
 		(start 97.2173 62.11)
-		(end 97.9517 62.8444)
+		(end 99 63.8927)
+		(width 0.5)
+		(layer "B.Cu")
+		(net "/LORA_SCK")
+	)
+	(segment
+		(start 99 63.8927)
+		(end 99 66.16)
+		(width 0.5)
+		(layer "B.Cu")
+		(net "/LORA_SCK")
+	)
+	(segment
+		(start 39.785 63.19)
+		(end 58.3341 63.19)
 		(width 0.5)
 		(layer "B.Cu")
@@
 		(width 0.5)
 		(layer "B.Cu")
-		(net "/LORA_SCK")
-	)
-	(segment
-		(start 39.785 63.19)
-		(end 58.3341 63.19)
-		(width 0.5)
-		(layer "B.Cu")
-		(net "/LORA_SCK")
-	)
-	(segment
-		(start 97.9517 67.2083)
-		(end 96.7 68.46)
-		(width 0.5)
-		(layer "B.Cu")
-		(net "/LORA_SCK")
-	)
-	(segment
-		(start 59.4141 62.11)
-		(end 97.2173 62.11)
-		(width 0.5)
-		(layer "B.Cu")
